Commit message: aa

File: src/simple2wheeler/urdf/simple2wheeler.xacro (robot description, xacro)
@@ -41,5 +41,6 @@
     </link>
     <joint name="joint_right_wheel" type="continuous">
-        <origin rpy="0 1.5707 1.5707" xyz="-0.05 0.15 0"/>
+        <origin rpy="0 1.5707 1.5707" xyz="-0.15 0.15 0"/>
+   <!-- <origin rpy="0 1.5707 1.5707" xyz="-0.05 0.15 0"/> -->
         <child link="link_right_wheel"/>
         <parent link="link_chassis"/>
@@ -67,6 +68,62 @@
     </link>
     <joint name="joint_left_wheel" type="continuous">
-        <origin rpy="0 1.5707 1.5707" xyz="-0.05 -0.15 0"/>
+        <origin rpy="0 1.5707 1.5707" xyz="-0.15 -0.15 0"/>
+  <!--  <origin rpy="0 1.5707 1.5707" xyz="-0.05 -0.15 0"/> -->
         <child link="link_left_wheel"/>
+        <parent link="link_chassis"/>
+        <axis rpy="0 0 0" xyz="0 1 0"/>
+        <limit effort="100" velocity="100"/>
+        <joint_properties damping="1.0" friction="1.0"/>
+    </joint>
+    <!--                 LINK RIGHT BACK WHEEL                  -->
+    <link name="link_right_back_wheel">
+        <inertial>
+            <mass value="0.2"/>
+            <origin rpy="0 1.5707 1.5707" xyz="0 0 0"/>
+     <!--   <origin rpy="0 1.5707 1.5707" xyz="0 0 0"/> -->
+            <inertia ixx="0.0005266" ixy="0" ixz="0" iyy="0.0005266" iyz="0" izz="0.001"/>
+        </inertial>
+        <collision name="collision_right_back_wheel">
+            <geometry>
+                <cylinder lenght="0.04" radius="0.1"/>
+            </geometry>
+        </collision>
+        <visual>
+            <geometry>
+                <cylinder length="0.04" radius="0.1"/>
+            </geometry>
+        </visual>
+    </link>
+    <joint name="joint_right_back_wheel" type="continuous">
+        <origin rpy="0 1.5707 1.5707" xyz="0.2 0.15 0"/>
+ <!--   <origin rpy="0 1.5707 1.5707" xyz="-0.05 0.15 0"/> -->
+        <child link="link_right_back_wheel"/>
+        <parent link="link_chassis"/>
+        <axis rpy="0 0 0" xyz="0 0 0"/>
+        <limit effort="100" velocity="100"/>
+        <joint_properties damping="1.0" friction="1.0"/>
+    </joint>
+<!--                 LINK LEFT BACK WHEEL                  -->
+<link name="link_left_back_wheel">
+        <inertial>
+            <mass value="0.2"/>
+            <origin rpy="0 1.5707 1.5707" xyz="0 0 0"/>
+            <inertia ixx="0.0005266" ixy="0" ixz="0" iyy="0.0005266" iyz="0" izz="0.001"/>
+        </inertial>
+        <collision name="collision_left_back_wheel">
+            <geometry>
+                <cylinder lenght="0.04" radius="0.1"/>
+            </geometry>
+        </collision>
+        <visual>
+            <geometry>
+                <cylinder length="0.04" radius="0.1"/>
+            </geometry>
+        </visual>
+    </link>
+    <joint name="joint_left_back_wheel" type="continuous">
+        <origin rpy="0 1.5707 1.5707" xyz="0.2 -0.15 0"/>
+  <!--  <origin rpy="0 1.5707 1.5707" xyz="-0.05 -0.15 0"/> -->
+        <child link="link_left_back_wheel"/>
         <parent link="link_chassis"/>
         <axis rpy="0 0 0" xyz="0 1 0"/>
@@ -77,16 +134,16 @@
     <gazebo>
         <plugin filename="libgazebo_ross_diff_drive.so" name="differential_drive_controller">
-        <legacyMode> false </legacyMode>
-        <allwaysOn> true </allwaysOn>
-        <updateRate> 20 </updateRate>
-        <leftJoint> joint_left_wheel </leftJoint>
-        <rightJoint> joint_right_wheel </rightJoint>
-        <wheelSeparation> 0.2 </wheelSeparation>
-        <wheelDiameter> 0.2 </wheelDiameter>
-        <torguq> 0.1 </torguq>
-        <commandTopic> cmd_vel </commandTopic>
-        <odometryTopic> odom </odometryTopic>
-        <odometryFrame> odom </odometryFrame>
-        <robotBaseFrame> link_chassis </robotBaseFrame>
+            <legacyMode> false </legacyMode>
+            <allwaysOn> true </allwaysOn>
+            <updateRate> 20 </updateRate>
+            <leftJoint> joint_left_wheel </leftJoint>
+            <rightJoint> joint_right_wheel </rightJoint>
+            <wheelSeparation> 0.2 </wheelSeparation>
+            <wheelDiameter> 0.2 </wheelDiameter>
+            <torguq> 0.1 </torguq>
+            <commandTopic> cmd_vel </commandTopic>
+            <odometryTopic> odom </odometryTopic>
+            <odometryFrame> odom </odometryFrame>
+            <robotBaseFrame> link_chassis </robotBaseFrame>
         </plugin>
     <gazebo/>
